Commit message: web_init

File: urdf/mano.urdf (robot description, URDF)
Before this commit: robot mano, 27 links, 26 joints
Links:
- removed link base_rx_link
- removed link base_ry_link
- removed link base_x_link
- removed link base_y_link
- removed link base_z_link
- removed link world_link
Joints:
- removed joint j_base_rx
- removed joint j_base_ry
- removed joint j_base_rz
- removed joint j_base_x
- removed joint j_base_y
- removed joint j_base_z
